File: skeem/RVP_TopeltKell.kicad_sch (KiCad schematic)
At the start: 30 parts, among them J1 Barrel_Jack, J10 Conn_01x03_Pin, J2 USB_B_Mini, J3 JST XH 5 pin, M1 Stepper_minute, M2 Stepper_hour, SW1 SW_BOOT, SW2 SW_RESET, U1 ESP32-S3-WROOM-1, U2 74HC4851, U3 LD1117S33TR_SOT223, U4 LD1117S50TR_SOT223, U5 CP2102N-Axx-xQFN24, U6 74HC4851, U7 74LVC2G53

Commit message: skem
Parts:
- removed C3, C5: 100n, symbol Device:C
- removed C4, C6: 10u, symbol Device:C
- removed J2: USB_B_Mini, symbol Connector:USB_B_Mini
- removed U2, U6: 74HC4851, symbol RVP_TopeltKell:74HC4851
- removed U3: LD1117S33TR_SOT223, Package_TO_SOT_SMD:SOT-223-3_TabPin2, symbol Regulator_Linear:LD1117S33TR_SOT223
- removed U4: LD1117S50TR_SOT223, Package_TO_SOT_SMD:SOT-223-3_TabPin2, symbol Regulator_Linear:LD1117S50TR_SOT223
- added J2: USB_B_Mini, symbol RVP_TopeltKell:USB_B_Mini
- added R7, R8: R, symbol Device:R
- added U2, U6: 74HCT4851, symbol RVP_TopeltKell:74HCT4851
- C7: value C -> 4.7
- C8: value C -> 0.1u
- R3: value R -> 4k7
Connections:
- net BOOT is gone; now on net ESP_BOOT: C1.2, SW1.2
- net RST is gone; now on net ESP_EN: C2.2, SW2.2
- net +3V3: no longer C1.1, C2.1, C7.1, C8.2, J1.2, J10.2 (Pin_2), R1.2, R2.2, R4.2, R5.2, R6.2, SW1.1, SW2.1, U5.2 (GND), U5.25 (GND), U7.3 (GND), U7.4 (GND)
- net +5V: now also J2.1 (VBUS), U2.16 (VCC), U6.16 (VCC)
- net SEL1: now also U2.11 (S0), U6.11 (S0)
- net SEL2: now also U2.10 (S1), U6.10 (S1)
- net SEL3: now also U2.9 (S2), U6.9 (S2)
- net SERVO0: now also U2.13 (Y0)
- net SERVO1: now also U2.14 (Y1)
- net SERVO2: now also U2.15 (Y2)
- net SERVO8: now also U6.13 (Y0)
- net SERVO9: now also U6.14 (Y1)
- net ESP_EN: now reaches U5.19 (~{RTS})
- net ESP_BOOT: now reaches U5.23 (~{DTR})
- net at U5.3 (D+): now also J2.3 (D+)
- net at U5.4 (D-): now also J2.2 (D-)
- net at R6.1: now also U6. (~{EN})
- net at U7.6 (Y1): now also R8.1, U6.3 (Z)
- net at U7.7 (Y0): now also R7.1, U2.3 (Z)
- net at R4.1: now also U2. (~{EN})
- new net GND: C1.1, C2.1, C7.1, C8.2, J1.2, J10.2 (Pin_2), J2.5 (GND), J2.6 (Shield), R1.2, R2.2, R4.2, R5.2, R6.2, R7.2, R8.2, SW1.1, SW2.1, U2. (~{EN}), U5.2 (GND), U5.25 (GND), U6. (~{EN}), U7.3 (GND), U7.4 (GND)
- new net SERVO10: U6.15 (Y2)
- new net SERVO11: U6.12 (Y3)
- new net SERVO3: U2.12 (Y3)
- new net SERVO4: U2.1 (Y4)
- new net SERVO5: U2.5 (Y5)
- new net SERVO6: U2.2 (Y6)
- new net SERVO7: U2.4 (Y7)
- no-connect marks 12 -> 14
Other:
- note added: "74HCT use TTL logic levels i.e can use SEL and Z with 3V3"
- note added: "KAS NEED SUUDAVAD PIISAVALT VOOLU V2LJA ANDA?"
- note added: "tee sellele suured padid, et k2sitsi joota saaks"
- note removed: "another LD1117 for 5V->3V3?"
- note removed: "kas neid saab juhtida 3.3, kui kasutan TTL kive? s.t 74HCT!"
- note removed: "kas siin on floating? uuri, kas on pull up vms"
- note removed: "neid on TTL"
- note removed: "pane v6imsused juurde"
- note removed: "seda kivi pole TTL aga pole vaja ka"
- moved on the sheet: C7, C8, J1, R2, R4, R5, R6, U7

Commit message: skeem edeneb
Parts:
- removed J10: Conn_01x03_Pin, Connector_PinHeader_2.54mm:PinHeader_1x03_P2.54mm_Vertical, symbol Connector:Conn_01x03_Pin
- removed J3: JST XH 5 pin, symbol Connector_Generic:Conn_01x05
- removed M1: Stepper_minute, symbol Motor:Stepper_Motor_bipolar
- removed M2: Stepper_hour, symbol Motor:Stepper_Motor_bipolar
- removed R4, R5, R6, R7, R8: R, symbol Device:R
- removed U2, U6: 74HCT4851, symbol RVP_TopeltKell:74HCT4851
- removed U7: 74LVC2G53, symbol RVP_TopeltKell:74LVC2G53
- added D2: PRTR5V0U2X, Package_TO_SOT_SMD:SOT-143, symbol Power_Protection:PRTR5V0U2X
- C7: value 4.7 -> 4.7u
Connections:
- net +5V: now also D2.4 (VCC)
- net GND: now also D2.1 (GND)
- new net D+: D2.3 (I/O2)
- new net D-: D2.2 (I/O1)
- no-connect marks 14 -> 10
Other:
- added sheet Servo (servo.kicad_sch)
- added sheet Stepper (Stepper.kicad_sch)
- note added: "! tee sellele suured padid, et k2sitsi joota saaks !"
- note added: "ESD protection"
- note added: "KUIDAS KAITSTA USBd TOITEADAPTERI YHENDAMISE EEST? St et arvuti ei plahvataks kui seinaadapter ja USB juhe korraga yhendatud"
- note added: "LOE KAARLI CHECKLISTI TEAMSIST"
- note removed: "12x servo pin header"
- note removed: "74HCT use TTL logic levels i.e can use SEL and Z with 3V3"
- note removed: "???"
- note removed: "ESD protection? tee nutipraxi j2rgi"
- note removed: "KAS NEED SUUDAVAD PIISAVALT VOOLU V2LJA ANDA?"
- note removed: "Servo control demultiplexing and level shifting"
- note removed: "Stepper drivers"
- note removed: "Stepper motors and servos"
- note removed: "leia ti.com mootor driver kivi"
- note removed: "loe kaarli nimekirja teamsis"
- note removed: "tee sellele suured padid, et k2sitsi joota saaks"
- moved on the sheet: C1, C2, C7, C8, D1, J1, J2, R1, R2, R3, SW1, SW2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
