File: skeem/RVP_TopeltKell.kicad_sch (KiCad schematic)
At the start: 15 parts, among them J1 Barrel_Jack, J2 USB_B_Mini, SW1 SW_BOOT, SW2 SW_RESET, U1 ESP32-S3-WROOM-1, U5 CP2102N-Axx-xQFN24

Commit message: Hall Sensor
Parts:
- added U8, U9: AH3761, Topeltkell:AH3761-WG-7, symbol RVP_TopeltKell:AH3761
Changed lines of the file:
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@@
+    )
+  )
+  (symbol (lib_id "RVP_TopeltKell:AH3761") (at 200.66 203.2 0) (unit 1)
+    (in_bom yes) (on_board yes) (dnp no) (fields_autoplaced)
+    (property "Reference" "U8" (at 210.82 198.12 0)
+      (effects (font (size 1.27 1.27)))
+    )
+    (property "Value" "AH3761" (at 210.82 200.66 0)
+      (effects (font (size 1.27 1.27)))
+    )
+    (property "Footprint" "Topeltkell:AH3761-WG-7" (at 220.98 231.14 0)
+      (effects (font (size 1.27 1.27)) hide)
+    )
+    (property "Datasheet" "https://www.farnell.com/datasheets/608727.pdf" (at 213.36 226.06 0)
+      (effects (font (size 1.27 1.27)) hide)
+    )
+    (pin "1")
+    (pin "2")
+    (pin "3")
+    (instances
+      (project "RVP_TopeltKell"
+        (path "/55c41515-c5b3-46de-9fdd-e6e788e90361"
+          (reference "U8") (unit 1)
+        )
+      )
     )
   )
@@
         )
       )
+    )
+  )
+  (symbol (lib_id "RVP_TopeltKell:AH3761") (at 236.22 203.2 0) (unit 1)
+    (in_bom yes) (on_board yes) (dnp no) (fields_autoplaced)
+    (property "Reference" "U9" (at 246.38 198.12 0)
+      (effects (font (size 1.27 1.27)))
+    )
+    (property "Value" "AH3761" (at 246.38 200.66 0)
+      (effects (font (size 1.27 1.27)))
+    )
+    (property "Footprint" "Topeltkell:AH3761-WG-7" (at 256.54 231.14 0)
+      (effects (font (size 1.27 1.27)) hide)
+    )
+    (property "Datasheet" "https://www.farnell.com/datasheets/608727.pdf" (at 248.92 226.06 0)
+      (effects (font (size 1.27 1.27)) hide)
+    )
+    (pin "1")
+    (pin "2")
+    (pin "3")
+    (instances
+      (project "RVP_TopeltKell"
+        (path "/55c41515-c5b3-46de-9fdd-e6e788e90361"
+          (reference "U9") (unit 1)
+        )
+      )

Commit message: power mgmt
Parts:
- added C4, C5: 100n, symbol Device:C
- added D3, D4: D_Zener, symbol Device:D_Zener
- added L1, L2: 3.3u, symbol Device:L
- added R10, R12: 10k, symbol Device:R
- added R11: 31k6, symbol Device:R
- added R9: 52k3, symbol Device:R
- added U10, U11: AP62300, symbol RVP_TopeltKell:AP62300
- C7: value 4.7u -> 4u7
- C8: value 0.1u -> 100n
Connections:
- net +3V3: now also L2.2, R11.1
- net +5V: now also L1.2, R9.1; no longer J2.1 (VBUS), U5.8 (VBUS)
- net +9V: now also D3.1 (K), D4.1 (K), U10.3 (VIN), U11.3 (VIN)
- net GND: now also R10.2, R12.2, U10.1 (GND), U11.1 (GND)
- new net: D4.2 (A), U11.5 (EN)
- new net: C4.1, L1.1, U10.2 (SW)
- new net: C4.2, U10.6 (BST)
- new net: R11.2, R12.1, U11.4 (FB)
- new net: C5.1, L2.1, U11.2 (SW)
- new net: C5.2, U11.6 (BST)
- new net: D3.2 (A), U10.5 (EN)
- new net: R10.1, R9.2, U10.4 (FB)
- new net VBUS: J2.1 (VBUS), U5.8 (VBUS)
Other:
- note added: "Programming only works with external power adapter connected"
- note added: "resistor divider values from datasheet"
- note removed: "LEIA SWITCH MODE POWER SUPPLY SMPS Buck converter ti.com lehelt :)"
- moved on the sheet: D1, D2, R1, U1

Commit message: arendus
Parts:
- added C10, C11, C12, C13: 22u, symbol Device:C
- added C6, C9: 10u, symbol Device:C
Connections:
- net +3V3: now also C12.1
- net +5V: now also C10.1
- net +9V: now also C6.1, C9.1
- net GND: now also C11.2, C13.2, C6.2, C9.2
- new net: C10.2, C11.1
- new net: C12.2, C13.1
Other:
- note added: "TSOT-26"
- note added: "kas ja milliseid zenereid kasutada? "Leave floating for automatic startup. The EN has a precision threshold of 1.2V for programing the UVLO." absolute max 6 V"
- note added: "kuidas saada selliste v22rtustega takistid?"
- moved on the sheet: C1, C2, D3, SW1, SW2, U1

Commit message: nu and impruvd
Parts:
- removed U8, U9: AH3761, Topeltkell:AH3761-WG-7, symbol RVP_TopeltKell:AH3761
- added C17: 100n, symbol Device:C
- added C18: 22u, symbol Device:C
- added C3: 1u, symbol Device:C
- added D5: LED, symbol Device:LED
- added D6: LED_DEGUG, symbol Device:LED
- added R15: 100, symbol Device:R
- added R4: R, symbol Device:R
- added R7, R8: 10k, symbol Device:R
- R1: value R -> 100
- R3: value 4k7 -> 1k
- U1: value ESP32-S3-WROOM-1 -> ESP32-S3-WROOM-1-N4
Connections:
- net RXD is gone; now on net ESP_TXD: U5.20 (RXD)
- net TXD is gone; now on net ESP_RXD: U5.21 (TXD)
- net +3V3: now also U1.2 (3V3), C17.1, C18.1, R7.1
- net DIR_HOUR: now also U1.32 (IO39)
- net DIR_MINUTE: now also U1.33 (IO40)
- net ESP_BOOT: now also U1.27 (IO0)
- net ESP_EN: now also U1.3 (EN), C3.1, R7.2
- net GND: now also U1.1 (GND), U1.40 (GND), U1.41 (EPAD), C17.2, C18.2, C3.2, R15.2, R4.2, R8.1
- net SEL0: now also U1.17 (IO9)
- net SEL1: now also U1.18 (IO10)
- net SEL2: now also U1.19 (IO11)
- net SEL3: now also U1.20 (IO12)
- net SERVO_PWM: now also U1.21 (IO13)
- net STEP_HOUR: now also U1.34 (IO41)
- net STEP_MINUTE: now also U1.35 (IO42)
- net VBUS: now also D5.2 (A)
- net at U1.15 (IO3): now also U1.16 (IO46), U1.26 (IO45), R8.2
- net M0_HOUR: now reaches U1.28 (IO35)
- net M1_HOUR: now reaches U1.29 (IO36)
- net M0_MINUTE: now reaches U1.30 (IO37)
- net M1_MINUTE: now reaches U1.31 (IO38)
- net ESP_RXD: now reaches U1.36 (RXD0)
- net ESP_TXD: now reaches U1.37 (TXD0)
- net at U1.39 (IO1): now also D6.2 (A)
- net HALL_HOUR: now reaches U1.4 (IO4)
- net HALL_MINUTE: now reaches U1.5 (IO5)
- new net: D5.1 (K), R4.1
- new net: D6.1 (K), R15.1
- no-connect marks 10 -> 24
Other:
- sheet Servo renamed Servo motors
- sheet Stepper renamed Stepper motors
- note added: "Programming only works with external power adapter connected :)"
- note added: "kas saab juhtmega v2lja viia (nt TO-92 pakend)"
- note added: "kuidas pulldown t88tab?"
- note removed: "Programming only works with external power adapter connected"
- moved on the sheet: C1, C10, C11, C12, C13, C2, C4, C5, C6, C7, C8, C9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

Commit message: veel skeemi
Parts:
- removed C1: 100n, symbol Device:C
- removed D3, D4: D_Zener, symbol Device:D_Zener
- removed R11: 31k6, symbol Device:R
- removed SW1: SW_BOOT, symbol Switch:SW_Push
- added R18: 51k, symbol Device:R
- added R19: 1.5k, symbol Device:R
- added R20: 4.3k, symbol Device:R
- R1, R15: value 100 -> 220
- R4: value R -> 470
- R9: value 52k3 -> 27k
Connections:
- net +3V3: now also C13.1, R9.1
- net +5V: now also C11.1, R18.1; no longer R9.1
- net D+: now also J2.3 (D+), U5.3 (D+)
- net D-: now also J2.2 (D-), U5.4 (D-)
- net GND: now also C10.2, C12.2
- net at R12.1, U11.4 (FB): now also R20.2
- net at R10.1, U10.4 (FB): now also R19.2; no longer R9.2
- new net: R18.2, R19.1
- new net: R20.1, R9.2
- no-connect marks 24 -> 26
Other:
- note removed: "KUIDAS KAITSTA USBd TOITEADAPTERI YHENDAMISE EEST? St et arvuti ei plahvataks kui seinaadapter ja USB juhe korraga yhendatud"
- note removed: "kas ja milliseid zenereid kasutada? "Leave floating for automatic startup. The EN has a precision threshold of 1.2V for programing the UVLO." absolute max 6 V"
- note removed: "kuidas pulldown t88tab?"
- note removed: "kuidas saada selliste v22rtustega takistid?"
- note removed: "resistor divider values from datasheet"
- moved on the sheet: C17, C18, C6, C7, C8, C9, D1, D2, D5, J2, R1, R10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

Commit message: skeem
Parts:
- U1: renamed from U10; footprint (none) -> Topeltkell:TSOT26
- U2: renamed from U11; footprint (none) -> Topeltkell:TSOT26
- renumbered C6 to C1, C8 to C10, C18 to C11, C17 to C12, C3 to C13, C2 to C14, C4 to C2, C10 to C3, C11 to C4, C9 to C5, C5 to C6, C12 to C7, C13 to C8, C7 to C9, D5 to D3, D6 to D4, R18 to R1, R4 to R10, R7 to R11, R8 to R12, R15 to R13, R19 to R2, R10 to R3, R9 to R4, R20 to R5, R12 to R6, R1 to R7, R3 to R8, R2 to R9, SW2 to SW1, U5 to U3, U1 to U4
Other:
- moved on the sheet: C1, C3, C4, C5

Commit message: skeem
Parts:
- added C24, C25, C26, C27: 100n, symbol Device:C
- added J17, J18: Conn_01x03_Pin, symbol Connector:Conn_01x03_Pin
- C2, C6: value 100n -> 330n
- L1: value 3.3u -> 4u7
- L2: value 3.3u -> 3u3; footprint (none) -> https://www.digikey.ee/en/products/detail/taiyo-yuden/NRS5030T3R3MMGJ/4157847
- R1: value 51k -> 52k3
- R2: value 1.5k -> 330
- R4: value 27k -> 31k6
- R5: value 4.3k -> 330
Connections:
- net +3V3: now also R2.2, R5.2, C26.2, J17.1 (Pin_1), J18.1 (Pin_1)
- net +5V: now also C24.2
- net +9V: now also C25.2, C27.2
- net GND: now also C24.1, C25.1, C26.1, C27.1, J17.2 (Pin_2), J18.2 (Pin_2)
- net HALL_HOUR: now also R2.1, J17.3 (Pin_3)
- net HALL_MINUTE: now also R5.1, J18.3 (Pin_3)
- net at R6.1, U2.4 (FB): now also R4.2; no longer R5.2
- net at R1.2: now also R3.1, U1.4 (FB); no longer R2.1
Other:
- sheet Servo motors ports: added SEL0, SEL1, SEL2, SEL3, SERVO_PWM; removed none
- sheet Stepper motors ports: added DIR_HOUR, DIR_MINUTE, M0_HOUR, M0_MINUTE, M1_HOUR, M1_MINUTE, STEP_HOUR, STEP_MINUTE; removed none
- note added: "3V3 net supplies: USB-UART chip ~10 mA ESP32 module 500 mA MUX0 ~100 mA 2x Hall latch 5 mA total max ~600 mA"
- note added: "4 kV human model w/o external components"
- note added: "5V net supplies: 2x Stepper motor ~500 mA 1x servo motor ~220 mA if not stalled 2x stepper driver ~20 mA 2x demux ~200 mA total max ~1000 mA"
- note added: "Extended ESD robustness necessary?"
- note added: "kui palju induktor voolu kannatab? uuri vali piisava current ratinguga vaata, et ei l2heks soojaks (takistus madal) saturation current, shielding siis otsusta"
- note added: "open drain output"
- note added: "panin induktorite datasheeti poe lingi"
- note added: "sensor datasheet"
- note removed: "kas saab juhtmega v2lja viia (nt TO-92 pakend)"
- moved on the sheet: C1, C10, C14, C2, C3, C4, C5, C6, C7, C8, C9, D1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

Commit message: skeem
Parts:
- J1: footprint (none) -> Connector_BarrelJack:BarrelJack_CLIFF_FC681465S_SMT_Horizontal
- J17, J18: footprint (none) -> Connector_PinHeader_2.54mm:PinHeader_1x03_P2.54mm_Vertical
- J2: footprint (none) -> Topeltkell:USB_Mini_B
- L2: footprint https://www.digikey.ee/en/products/detail/taiyo-yuden/NRS5030T3R3MMGJ/4157847 -> (none)
- R1, R10, R11, R12, R13, R2, R3, R4, R5, R6, R7, R8, R9: footprint (none) -> Resistor_SMD:R_0603_1608Metric_Pad0.98x0.95mm_HandSolder
- SW1: footprint (none) -> Button_Switch_SMD:SW_SPST_EVQQ2
- U1, U2: value AP62300 -> AP62200
Other:
- note added: "2.1 mm pin inner diameter"
- note added: "piisav current rating piisavalt madal takistus piisavalt suur saturation current shielded (me ei taha müra; ruum ja hind ei ole probleem)"
- note removed: "kui palju induktor voolu kannatab? uuri vali piisava current ratinguga vaata, et ei l2heks soojaks (takistus madal) saturation current, shielding siis otsusta"
- moved on the sheet: R13
Changed lines of the file:
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@@
     (stroke (width 0) (type default))
   )
-  (wire (pts (xy 255.27 121.92) (xy 259.08 121.92))
+  (wire (pts (xy 254 121.92) (xy 259.08 121.92))
     (stroke (width 0) (type default))
   )
@@
     (stroke (width 0) (type default))
   )
-  (wire (pts (xy 247.65 121.92) (xy 241.3 121.92))
+  (wire (pts (xy 246.38 121.92) (xy 241.3 121.92))
     (stroke (width 0) (type default))
   )
@@
     (effects (font (size 1.27 1.27)) (justify left bottom))
   )
-  (text "kui palju induktor voolu kannatab?\nuuri\nvali piisava current ratinguga\nvaata, et ei l2heks soojaks (takistus madal)\nsaturation current, shielding\nsiis otsusta"
-    (at 109.22 91.44 0)
+  (text "piisav current rating\npiisavalt madal takistus\npiisavalt suur saturation current \nshielded (me ei taha müra; ruum ja hind ei ole probleem)"
+    (at 107.95 88.9 0)
     (effects (font (size 1.27 1.27)) (justify left bottom))
   )
@@
     (effects (font (size 5.08 5.08)) (justify left bottom))
   )
-  (text "MWL001125 AC/DC 9V 1.33A wall adapter" (at 21.59 25.4 0)
+  (text "2.1 mm pin inner diameter" (at 21.59 26.67 0)
+    (effects (font (size 1.27 1.27)) (justify left bottom))
+  )
+  (text "MWL001125 AC/DC 9V 1.33A wall adapter" (at 21.59 24.13 0)
     (effects (font (size 1.27 1.27)) (justify left bottom))
   )
@@
   )
   (text "3V3 net supplies:\n\nUSB-UART chip ~10 mA\nESP32 module 500 mA\nMUX0 ~100 mA\n2x Hall latch 5 mA\n\ntotal max ~600 mA"
-    (at 148.59 109.22 0)
+    (at 147.32 110.49 0)
     (effects (font (size 1.27 1.27)) (justify left bottom))
   )
   (text "5V net supplies:\n\n2x Stepper motor ~500 mA\n1x servo motor ~220 mA if not stalled\n2x stepper driver ~20 mA\n2x demux ~200 mA\n\ntotal max ~1000 mA"
-    (at 148.59 73.66 0)
+    (at 148.59 76.2 0)
     (effects (font (size 1.27 1.27)) (justify left bottom))
   )
@@
       (effects (font (size 1.27 1.27)) (justify left))
     )
-    (property "Footprint" "" (at 98.552 111.76 90)
+    (property "Footprint" "Resistor_SMD:R_0603_1608Metric_Pad0.98x0.95mm_HandSolder" (at 98.552 111.76 90)
       (effects (font (size 1.27 1.27)) hide)
     )
@@
       (effects (font (size 1.27 1.27)) (justify right))
     )
-    (property "Footprint" "" (at 184.658 200.66 90)
+    (property "Footprint" "Resistor_SMD:R_0603_1608Metric_Pad0.98x0.95mm_HandSolder" (at 184.658 200.66 90)
       (effects (font (size 1.27 1.27)) hide)
     )
@@
       (effects (font (size 1.27 1.27)))
     )
-    (property "Value" "AP62300" (at 71.12 88.9 0)
+    (property "Value" "AP62200" (at 71.12 88.9 0)
       (effects (font (size 1.27 1.27)))
     )
@@
       (effects (font (size 1.27 1.27)))
     )
-    (property "Footprint" "" (at 252.73 91.948 90)
+    (property "Footprint" "Resistor_SMD:R_0603_1608Metric_Pad0.98x0.95mm_HandSolder" (at 252.73 91.948 90)
       (effects (font (size 1.27 1.27)) hide)
     )
@@
       (effects (font (size 1.27 1.27)) (justify right))
     )
-    (property "Footprint" "" (at 236.728 200.66 90)
+    (property "Footprint" "Resistor_SMD:R_0603_1608Metric_Pad0.98x0.95mm_HandSolder" (at 236.728 200.66 90)
       (effects (font (size 1.27 1.27)) hide)
     )
@@
       (effects (font (size 1.27 1.27)))
     )
-    (property "Footprint" "" (at 100.33 152.908 90)
+    (property "Footprint" "Resistor_SMD:R_0603_1608Metric_Pad0.98x0.95mm_HandSolder" (at 100.33 152.908 90)
       (effects (font (size 1.27 1.27)) hide)
     )
@@
     )
   )
-  (symbol (lib_id "Device:R") (at 251.46 121.92 270) (mirror x) (unit 1)
+  (symbol (lib_id "Device:R") (at 250.19 121.92 270) (mirror x) (unit 1)
     (in_bom yes) (on_board yes) (dnp no)
-    (property "Reference" "R13" (at 251.46 119.38 90)
-      (effects (font (size 1.27 1.27)))
-    )
-    (property "Value" "220" (at 251.46 121.92 90)
-      (effects (font (size 1.27 1.27)))
-    )
-    (property "Footprint" "" (at 251.46 123.698 90)
-      (effects (font (size 1.27 1.27)) hide)
-    )
-    (property "Datasheet" "~" (at 251.46 121.92 0)
+    (property "Reference" "R13" (at 250.19 119.38 90)
+      (effects (font (size 1.27 1.27)))
+    )
+    (property "Value" "220" (at 250.19 121.92 90)
+      (effects (font (size 1.27 1.27)))
+    )
+    (property "Footprint" "Resistor_SMD:R_0603_1608Metric_Pad0.98x0.95mm_HandSolder" (at 250.19 123.698 90)
+      (effects (font (size 1.27 1.27)) hide)
+    )
+    (property "Datasheet" "~" (at 250.19 121.92 0)
       (effects (font (size 1.27 1.27)) hide)
     )
@@
       (effects (font (size 1.27 1.27)) (justify left))
     )
-    (property "Footprint" "" (at 98.552 69.85 90)
+    (property "Footprint" "Resistor_SMD:R_0603_1608Metric_Pad0.98x0.95mm_HandSolder" (at 98.552 69.85 90)
       (effects (font (size 1.27 1.27)) hide)
     )
@@
       (effects (font (size 1.27 1.27)))
     )
-    (property "Footprint" "" (at 123.19 38.608 90)
+    (property "Footprint" "Resistor_SMD:R_0603_1608Metric_Pad0.98x0.95mm_HandSolder" (at 123.19 38.608 90)
       (effects (font (size 1.27 1.27)) hide)
     )
@@
       (effects (font (size 1.27 1.27)))
     )
-    (property "Footprint" "" (at 137.16 175.768 90)
+    (property "Footprint" "Resistor_SMD:R_0603_1608Metric_Pad0.98x0.95mm_HandSolder" (at 137.16 175.768 90)
       (effects (font (size 1.27 1.27)) hide)
     )
@@
       (effects (font (size 1.27 1.27)) (justify right))
     )
-    (property "Footprint" "" (at 209.55 199.39 0)
+    (property "Footprint" "Connector_PinHeader_2.54mm:PinHeader_1x03_P2.54mm_Vertical" (at 209.55 199.39 0)
       (effects (font (size 1.27 1.27)) hide)
     )
@@
   (symbol (lib_id "RVP_TopeltKell:USB_B_Mini") (at 29.21 158.75 0) (unit 1)
     (in_bom yes) (on_board yes) (dnp no)
-    (property "Reference" "J2" (at 33.02 160.02 0)
-      (effects (font (size 1.27 1.27)))
-    )
-    (property "Value" "USB_B_Mini" (at 30.48 170.18 90)
-      (effects (font (size 1.27 1.27)))
-    )
-    (property "Footprint" "" (at 29.21 158.75 0)
-      (effects (font (size 1.27 1.27)) hide)
-    )
-    (property "Datasheet" "" (at 29.21 158.75 0)
+    (property "Reference" "J2" (at 30.48 157.48 0)
+      (effects (font (size 1.27 1.27)))
+    )
+    (property "Value" "USB_B_Mini" (at 27.94 168.91 90)
+      (effects (font (size 1.27 1.27)))
+    )
+    (property "Footprint" "Topeltkell:USB_Mini_B" (at 29.21 158.75 0)
+      (effects (font (size 1.27 1.27)) hide)
+    )
+    (property "Datasheet" "https://www.farnell.com/datasheets/2374176.pdf" (at 29.21 158.75 0)
       (effects (font (size 1.27 1.27)) hide)
     )
@@
       (effects (font (size 1.27 1.27)))
     )
-    (property "Footprint" "" (at 215.9 63.5 0)
+    (property "Footprint" "Button_Switch_SMD:SW_SPST_EVQQ2" (at 215.9 63.5 0)
       (effects (font (size 1.27 1.27)) hide)
     )
@@
       (effects (font (size 1.27 1.27)) (justify left))
     )
-    (property "Footprint" "" (at 98.552 104.14 90)
+    (property "Footprint" "Resistor_SMD:R_0603_1608Metric_Pad0.98x0.95mm_HandSolder" (at 98.552 104.14 90)
       (effects (font (size 1.27 1.27)) hide)
     )
@@
       (effects (font (size 1.27 1.27)))
     )
-    (property "Footprint" "https://www.digikey.ee/en/products/detail/taiyo-yuden/NRS5030T3R3MMGJ/4157847" (at 93.98 100.33 0)
+    (property "Footprint" "" (at 93.98 100.33 0)
       (effects (font (size 1.27 1.27)) hide)
     )
@@
       (effects (font (size 1.27 1.27)))
     )
-    (property "Footprint" "" (at 50.8 197.358 90)
+    (property "Footprint" "Resistor_SMD:R_0603_1608Metric_Pad0.98x0.95mm_HandSolder" (at 50.8 197.358 90)
       (effects (font (size 1.27 1.27)) hide)
     )
@@
       (effects (font (size 1.27 1.27)) (justify right))
     )
-    (property "Footprint" "" (at 261.62 199.39 0)
+    (property "Footprint" "Connector_PinHeader_2.54mm:PinHeader_1x03_P2.54mm_Vertical" (at 261.62 199.39 0)
       (effects (font (size 1.27 1.27)) hide)
     )
@@
       (effects (font (size 1.27 1.27)))
     )
-    (property "Value" "AP62300" (at 71.12 54.61 0)
+    (property "Value" "AP62200" (at 71.12 54.61 0)
       (effects (font (size 1.27 1.27)))
     )
@@
       (effects (font (size 1.27 1.27)))
     )
-    (property "Footprint" "" (at 29.21 36.576 0)
+    (property "Footprint" "Connector_BarrelJack:BarrelJack_CLIFF_FC681465S_SMT_Horizontal" (at 29.21 36.576 0)
       (effects (font (size 1.27 1.27)) hide)
     )
@@
       (effects (font (size 1.27 1.27)) (justify left))
     )
-    (property "Footprint" "" (at 98.552 77.47 90)
+    (property "Footprint" "Resistor_SMD:R_0603_1608Metric_Pad0.98x0.95mm_HandSolder" (at 98.552 77.47 90)
       (effects (font (size 1.27 1.27)) hide)
     )
@@
       (effects (font (size 1.27 1.27)) (justify left))
     )
-    (property "Footprint" "" (at 253.492 48.26 90)
-      (effects (font (size 1.27 1.27)) hide)
-    )
+    (property "Footprint" "Resistor_SMD:R_0603_1608Metric_Pad0.98x0.95mm_HandSolder" (at 253.492 48.26 90)
+      (effects (font (size 1.27 1.27)) hide)
+    )
