File: skeem/RVP_TopeltKell.kicad_sch (KiCad schematic)
At the start: 46 parts, among them J1 Barrel_Jack, J17 Conn_01x03_Pin, J18 Conn_01x03_Pin, J2 USB_B_Mini, SW1 SW_RESET, U1 AP62200, U2 AP62200, U3 CP2102N-Axx-xQFN24, U4 ESP32-S3-WROOM-1-N4

Commit message: pcb comp placement draft
Parts:
- removed J17, J18: Conn_01x03_Pin, Connector_PinHeader_2.54mm:PinHeader_1x03_P2.54mm_Vertical, symbol Connector:Conn_01x03_Pin
- removed R5: 330, Resistor_SMD:R_0603_1608Metric_Pad0.98x0.95mm_HandSolder, symbol Device:R
- removed U1, U2: AP62200, Topeltkell:TSOT26, symbol RVP_TopeltKell:AP62300
- added H1, H2, H3, H4: MountingHole, MountingHole:MountingHole_3.2mm_M3, symbol Mechanical:MountingHole
- added R17, R4: 10k, Resistor_SMD:R_0603_1608Metric_Pad0.98x0.95mm_HandSolder, symbol Device:R
- added R2: 47k, Resistor_SMD:R_0603_1608Metric_Pad0.98x0.95mm_HandSolder, symbol Device:R
- added U1, U2: AP62200, Topeltkell:TSOT26, symbol RVP_TopeltKell:AP62200
- added U5, U6: TLV4961, Package_TO_SOT_THT:TO-92S, symbol RVP_TopeltKell:TLV4961
- C1: footprint (none) -> Capacitor_SMD:C_0805_2012Metric_Pad1.18x1.45mm_HandSolder
- C10: renamed from C7; footprint (none) -> Capacitor_SMD:C_1206_3216Metric_Pad1.33x1.80mm_HandSolder
- C11: renamed from C8; footprint (none) -> Capacitor_SMD:C_1206_3216Metric_Pad1.33x1.80mm_HandSolder
- C12: renamed from C26; footprint (none) -> Capacitor_SMD:C_0603_1608Metric_Pad1.08x0.95mm_HandSolder
- C13: renamed from C9; footprint (none) -> Capacitor_SMD:C_0805_2012Metric_Pad1.18x1.45mm_HandSolder
- C14: renamed from C10; footprint (none) -> Capacitor_SMD:C_0603_1608Metric_Pad1.08x0.95mm_HandSolder
- C15: renamed from C11; footprint (none) -> Capacitor_SMD:C_1206_3216Metric_Pad1.33x1.80mm_HandSolder
- C16: renamed from C12; footprint (none) -> Capacitor_SMD:C_0603_1608Metric_Pad1.08x0.95mm_HandSolder
- C17: renamed from C13; footprint (none) -> Capacitor_SMD:C_0805_2012Metric_Pad1.18x1.45mm_HandSolder
- C18: renamed from C14; footprint (none) -> Capacitor_SMD:C_0603_1608Metric_Pad1.08x0.95mm_HandSolder
- C2: renamed from C25; footprint (none) -> Capacitor_SMD:C_0603_1608Metric_Pad1.08x0.95mm_HandSolder
- C3: renamed from C2; footprint (none) -> Capacitor_SMD:C_0603_1608Metric_Pad1.08x0.95mm_HandSolder
- C4: renamed from C3; footprint (none) -> Capacitor_SMD:C_1206_3216Metric_Pad1.33x1.80mm_HandSolder
- C5: renamed from C4; footprint (none) -> Capacitor_SMD:C_1206_3216Metric_Pad1.33x1.80mm_HandSolder
- C6: renamed from C24; footprint (none) -> Capacitor_SMD:C_0603_1608Metric_Pad1.08x0.95mm_HandSolder
- C7: renamed from C5; footprint (none) -> Capacitor_SMD:C_0805_2012Metric_Pad1.18x1.45mm_HandSolder
- C8: renamed from C27; footprint (none) -> Capacitor_SMD:C_0603_1608Metric_Pad1.08x0.95mm_HandSolder
- C9: renamed from C6; footprint (none) -> Capacitor_SMD:C_0603_1608Metric_Pad1.08x0.95mm_HandSolder
- D1: value LED -> LED_POWER; footprint (none) -> LED_SMD:LED_0603_1608Metric_Pad1.05x0.95mm_HandSolder
- D3: value LED -> LED_USB; footprint (none) -> LED_SMD:LED_0603_1608Metric_Pad1.05x0.95mm_HandSolder
- D4: footprint (none) -> LED_SMD:LED_0603_1608Metric_Pad1.05x0.95mm_HandSolder
- L1: footprint (none) -> Inductor_SMD:L_Wuerth_WE-PD-Typ-7345
- L2: footprint (none) -> Inductor_SMD:L_7.3x7.3_H3.5
- R10: renamed from R8; value 1k -> 10k
- R16: renamed from R2; value 330 -> 10k
- renumbered R7 to R1, R9 to R11, R10 to R12, R11 to R13, R12 to R14, R13 to R15, R1 to R3, R3 to R5, R4 to R7, R6 to R9
Connections:
- net +3V3: now also R17.2, U5.1 (VDD), U6.1 (VDD)
- net +9V: now also R2.1, U1.3 (VIN), U2.3 (VIN)
- net GND: now also R4.2, U1.1 (GND), U2.1 (GND), U5.2 (GND), U6.2 (GND)
- net HALL_HOUR: now also U5.3 (Q)
- net HALL_MINUTE: now also R17.1, U6.3 (Q)
- net at C3.1, L1.1: now also U1.2 (SW)
- net at C3.2: now also U1.6 (BST)
- net FB_3V3: now reaches R7.2, R9.1
- net FB_3V3: now also U2.4 (FB)
- net at C9.1, L2.1: now also U2.2 (SW)
- net at C9.2: now also U2.6 (BST)
- net FB_5V: now reaches R3.2, R5.1
- net FB_5V: now also U1.4 (FB)
- new net EN_DCDC: R2.2, R4.1, U1.5 (EN), U2.5 (EN)
- no-connect marks 26 -> 24
Other:
- note removed: "! tee sellele suured padid, et k2sitsi joota saaks !"
- note removed: "4 kV human model w/o external components"
- note removed: "Extended ESD robustness necessary?"
- note removed: "LOE KAARLI CHECKLISTI TEAMSIST"
- note removed: "open drain output"
- note removed: "panin induktorite datasheeti poe lingi"
- note removed: "piisav current rating piisavalt madal takistus piisavalt suur saturation current shielded (me ei taha müra; ruum ja hind ei ole probleem)"
- note removed: "sensor datasheet"
- moved on the sheet: C1, C2, C7, C8, J1, R16

Commit message: natuke pcbd
Parts:
- removed H4: MountingHole, MountingHole:MountingHole_3.2mm_M3, symbol Mechanical:MountingHole
- added R8: 470, Resistor_SMD:R_0603_1608Metric_Pad0.98x0.95mm_HandSolder, symbol Device:R
Connections:
- net +5V: no longer D2.4 (VCC)
- net D+: now also D2.2 (I/O1); no longer D2.3 (I/O2)
- net D-: now also D2.3 (I/O2); no longer D2.2 (I/O1)
- net GND: now also R8.2; no longer C18.1, SW1.1
- net VBUS: now also D2.4 (VCC)
- new net: C18.1, R8.1, SW1.1
Other:
- note added: "ARVUTA VOOLUSID (USB) JA PINGEJAGUR (ESB EN)"
Changed lines of the file:
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@@
   (junction (at 100.33 73.66) (diameter 0) (color 0 0 0 0)
   )
+  (junction (at 220.98 68.58) (diameter 0) (color 0 0 0 0)
+  )
   (junction (at 227.33 196.85) (diameter 0) (color 0 0 0 0)
   )
@@
   )
   (junction (at 124.46 100.33) (diameter 0) (color 0 0 0 0)
-  )
-  (junction (at 220.98 68.58) (diameter 0) (color 0 0 0 0)
   )
   (junction (at 36.195 58.42) (diameter 0) (color 0 0 0 0)
@@
     (stroke (width 0) (type default))
   )
-  (wire (pts (xy 224.79 68.58) (xy 220.98 68.58))
-    (stroke (width 0) (type default))
-  )
   (wire (pts (xy 130.81 153.67) (xy 143.51 153.67))
     (stroke (width 0) (type default))
@@
   )
   (wire (pts (xy 313.69 105.41) (xy 299.72 105.41))
+    (stroke (width 0) (type default))
+  )
+  (wire (pts (xy 228.6 68.58) (xy 231.775 68.58))
     (stroke (width 0) (type default))
   )
@@
     (effects (font (size 2.032 2.032)) (justify left bottom))
   )
+  (text "ARVUTA VOOLUSID (USB) JA PINGEJAGUR (ESB EN)" (at 197.485 86.36 0)
+    (effects (font (size 1.27 1.27)) (justify left bottom))
+  )
   (text "Power LED" (at 107.95 25.4 0)
     (effects (font (size 1.27 1.27)) (justify left bottom))
@@
     (effects (font (size 1.27 1.27)) (justify right bottom))
   )
-  (label "D-" (at 55.88 166.37 0) (fields_autoplaced)
-    (effects (font (size 1.27 1.27)) (justify left bottom))
+  (label "D-" (at 91.44 166.37 180) (fields_autoplaced)
+    (effects (font (size 1.27 1.27)) (justify right bottom))
   )
   (label "ESP_TXD" (at 256.54 67.31 0) (fields_autoplaced)
@@
     (effects (font (size 1.27 1.27)) (justify left bottom))
   )
-  (label "D+" (at 91.44 166.37 180) (fields_autoplaced)
-    (effects (font (size 1.27 1.27)) (justify right bottom))
+  (label "D+" (at 55.88 166.37 0) (fields_autoplaced)
+    (effects (font (size 1.27 1.27)) (justify left bottom))
   )
   (label "D+" (at 46.99 168.91 180) (fields_autoplaced)
@@
         (path "/55c41515-c5b3-46de-9fdd-e6e788e90361"
           (reference "#PWR03") (unit 1)
+        )
+      )
+    )
+  )
+  (symbol (lib_id "Device:R") (at 224.79 68.58 90) (unit 1)
+    (in_bom yes) (on_board yes) (dnp no)
+    (property "Reference" "R8" (at 224.79 66.04 90)
+      (effects (font (size 1.27 1.27)))
+    )
+    (property "Value" "470" (at 224.79 68.58 90)
+      (effects (font (size 1.27 1.27)))
+    )
+    (property "Footprint" "Resistor_SMD:R_0603_1608Metric_Pad0.98x0.95mm_HandSolder" (at 224.79 70.358 90)
+      (effects (font (size 1.27 1.27)) hide)
+    )
+    (property "Datasheet" "~" (at 224.79 68.58 0)
+      (effects (font (size 1.27 1.27)) hide)
+    )
+    (pin "1")
+    (pin "2")
+    (instances
+      (project "RVP_TopeltKell"
+        (path "/55c41515-c5b3-46de-9fdd-e6e788e90361"
+          (reference "R8") (unit 1)
         )
       )
@@
     )
   )
-  (symbol (lib_id "power:+5V") (at 73.66 153.67 0) (unit 1)
-    (in_bom yes) (on_board yes) (dnp no) (fields_autoplaced)
-    (property "Reference" "#PWR029" (at 73.66 157.48 0)
-      (effects (font (size 1.27 1.27)) hide)
-    )
-    (property "Value" "+5V" (at 73.66 148.59 0)
-      (effects (font (size 1.27 1.27)))
-    )
-    (property "Footprint" "" (at 73.66 153.67 0)
-      (effects (font (size 1.27 1.27)) hide)
-    )
-    (property "Datasheet" "" (at 73.66 153.67 0)
-      (effects (font (size 1.27 1.27)) hide)
-    )
-    (pin "1")
-    (instances
-      (project "RVP_TopeltKell"
-        (path "/55c41515-c5b3-46de-9fdd-e6e788e90361"
-          (reference "#PWR029") (unit 1)
-        )
-      )
-    )
-  )
   (symbol (lib_id "Device:R") (at 100.33 69.85 0) (unit 1)
     (in_bom yes) (on_board yes) (dnp no)
@@
         (path "/55c41515-c5b3-46de-9fdd-e6e788e90361"
           (reference "C4") (unit 1)
+        )
+      )
+    )
+  )
+  (symbol (lib_id "power:VBUS") (at 73.66 153.67 0) (unit 1)
+    (in_bom yes) (on_board yes) (dnp no) (fields_autoplaced)
+    (property "Reference" "#PWR022" (at 73.66 157.48 0)
+      (effects (font (size 1.27 1.27)) hide)
+    )
+    (property "Value" "VBUS" (at 73.66 148.59 0)
+      (effects (font (size 1.27 1.27)))
+    )
+    (property "Footprint" "" (at 73.66 153.67 0)
+      (effects (font (size 1.27 1.27)) hide)
+    )
+    (property "Datasheet" "" (at 73.66 153.67 0)
+      (effects (font (size 1.27 1.27)) hide)
+    )
+    (pin "1")
+    (instances
+      (project "RVP_TopeltKell"
+        (path "/55c41515-c5b3-46de-9fdd-e6e788e90361"
+          (reference "#PWR022") (unit 1)
         )
       )
@@
     )
   )
-  (symbol (lib_id "power:GND") (at 224.79 68.58 0) (mirror y) (unit 1)
-    (in_bom yes) (on_board yes) (dnp no) (fields_autoplaced)
-    (property "Reference" "#PWR011" (at 224.79 74.93 0)
-      (effects (font (size 1.27 1.27)) hide)
-    )
-    (property "Value" "GND" (at 224.79 73.66 0)
-      (effects (font (size 1.27 1.27)))
-    )
-    (property "Footprint" "" (at 224.79 68.58 0)
-      (effects (font (size 1.27 1.27)) hide)
-    )
-    (property "Datasheet" "" (at 224.79 68.58 0)
+  (symbol (lib_id "power:GND") (at 231.775 68.58 0) (mirror y) (unit 1)
+    (in_bom yes) (on_board yes) (dnp no) (fields_autoplaced)
+    (property "Reference" "#PWR011" (at 231.775 74.93 0)
+      (effects (font (size 1.27 1.27)) hide)
+    )
+    (property "Value" "GND" (at 231.775 73.66 0)
+      (effects (font (size 1.27 1.27)) hide)
+    )
+    (property "Footprint" "" (at 231.775 68.58 0)
+      (effects (font (size 1.27 1.27)) hide)
+    )
+    (property "Datasheet" "" (at 231.775 68.58 0)
       (effects (font (size 1.27 1.27)) hide)
     )
@@
         )
       )
-    )
-  )
-  (symbol (lib_id "Mechanical:MountingHole") (at 34.925 267.335 0) (unit 1)
-    (in_bom yes) (on_board yes) (dnp no) (fields_autoplaced)
-    (property "Reference" "H4" (at 38.1 266.065 0)
-      (effects (font (size 1.27 1.27)) (justify left))
-    )
-    (property "Value" "MountingHole" (at 38.1 268.605 0)
-      (effects (font (size 1.27 1.27)) (justify left))
-    )
-    (property "Footprint" "MountingHole:MountingHole_3.2mm_M3" (at 34.925 267.335 0)
-      (effects (font (size 1.27 1.27)) hide)
-    )
-    (property "Datasheet" "~" (at 34.925 267.335 0)
-      (effects (font (size 1.27 1.27)) hide)
-    )
-    (instances
-      (project "RVP_TopeltKell"
-        (path "/55c41515-c5b3-46de-9fdd-e6e788e90361"
-          (reference "H4") (unit 1)
-        )
-      )

Commit message: asi
Connections:
- net DIR_HOUR: now also U4.28 (IO35); no longer U4.32 (IO39)
- net DIR_MINUTE: now also U4.35 (IO42); no longer U4.33 (IO40)
- net M0_HOUR: now also U4.31 (IO38); no longer U4.28 (IO35)
- net M0_MINUTE: now also U4.32 (IO39); no longer U4.30 (IO37)
- net M1_HOUR: now also U4.30 (IO37); no longer U4.29 (IO36)
- net M1_MINUTE: now also U4.33 (IO40); no longer U4.31 (IO38)
- net STEP_HOUR: now also U4.29 (IO36); no longer U4.34 (IO41)
- net STEP_MINUTE: now also U4.34 (IO41); no longer U4.35 (IO42)
Other:
- note removed: "ARVUTA VOOLUSID (USB) JA PINGEJAGUR (ESB EN)"
- moved on the sheet: R8
Changed lines of the file:
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@@
     (stroke (width 0) (type default))
   )
-  (wire (pts (xy 299.72 116.84) (xy 314.96 116.84))
+  (wire (pts (xy 299.72 116.84) (xy 314.325 116.84))
     (stroke (width 0) (type default))
   )
@@
     (stroke (width 0) (type default))
   )
+  (wire (pts (xy 222.25 68.58) (xy 220.98 68.58))
+    (stroke (width 0) (type default))
+  )
   (wire (pts (xy 227.33 52.07) (xy 238.76 52.07))
     (stroke (width 0) (type default))
@@
     (stroke (width 0) (type default))
   )
-  (wire (pts (xy 228.6 68.58) (xy 231.775 68.58))
+  (wire (pts (xy 229.87 68.58) (xy 231.775 68.58))
     (stroke (width 0) (type default))
   )
@@
     (effects (font (size 2.032 2.032)) (justify left bottom))
   )
-  (text "ARVUTA VOOLUSID (USB) JA PINGEJAGUR (ESB EN)" (at 197.485 86.36 0)
-    (effects (font (size 1.27 1.27)) (justify left bottom))
-  )
   (text "Power LED" (at 107.95 25.4 0)
     (effects (font (size 1.27 1.27)) (justify left bottom))
@@
     (effects (font (size 1.27 1.27)) (justify left bottom))
   )
-  (label "M0_MINUTE" (at 313.69 97.79 180) (fields_autoplaced)
+  (label "M0_MINUTE" (at 313.69 105.41 180) (fields_autoplaced)
     (effects (font (size 1.27 1.27)) (justify right bottom))
   )
@@
     (effects (font (size 1.27 1.27)) (justify left bottom))
   )
-  (label "M1_HOUR" (at 313.69 93.98 180) (fields_autoplaced)
+  (label "M1_HOUR" (at 313.69 97.79 180) (fields_autoplaced)
     (effects (font (size 1.27 1.27)) (justify right bottom))
   )
@@
     (effects (font (size 1.27 1.27)) (justify left bottom))
   )
-  (label "DIR_MINUTE" (at 313.69 109.22 180) (fields_autoplaced)
+  (label "DIR_MINUTE" (at 314.325 116.84 180) (fields_autoplaced)
     (effects (font (size 1.27 1.27)) (justify right bottom))
   )
@@
     (effects (font (size 1.27 1.27)) (justify right bottom))
   )
-  (label "M1_MINUTE" (at 313.69 101.6 180) (fields_autoplaced)
+  (label "M1_MINUTE" (at 313.69 109.22 180) (fields_autoplaced)
     (effects (font (size 1.27 1.27)) (justify right bottom))
   )
@@
     (effects (font (size 1.27 1.27)) (justify left bottom))
   )
-  (label "STEP_MINUTE" (at 314.96 116.84 180) (fields_autoplaced)
-    (effects (font (size 1.27 1.27)) (justify right bottom))
-  )
-  (label "STEP_HOUR" (at 313.69 113.03 180) (fields_autoplaced)
+  (label "STEP_MINUTE" (at 313.69 113.03 180) (fields_autoplaced)
+    (effects (font (size 1.27 1.27)) (justify right bottom))
+  )
+  (label "STEP_HOUR" (at 313.69 93.98 180) (fields_autoplaced)
     (effects (font (size 1.27 1.27)) (justify right bottom))
   )
@@
     (effects (font (size 1.27 1.27)) (justify right bottom))
   )
-  (label "M0_HOUR" (at 313.69 90.17 180) (fields_autoplaced)
+  (label "M0_HOUR" (at 313.69 101.6 180) (fields_autoplaced)
     (effects (font (size 1.27 1.27)) (justify right bottom))
   )
@@
     (effects (font (size 1.27 1.27)) (justify left bottom))
   )
-  (label "DIR_HOUR" (at 313.69 105.41 180) (fields_autoplaced)
+  (label "DIR_HOUR" (at 313.69 90.17 180) (fields_autoplaced)
     (effects (font (size 1.27 1.27)) (justify right bottom))
   )
@@
     )
   )
-  (symbol (lib_id "Device:R") (at 224.79 68.58 90) (unit 1)
+  (symbol (lib_id "Device:R") (at 226.06 68.58 90) (unit 1)
     (in_bom yes) (on_board yes) (dnp no)
-    (property "Reference" "R8" (at 224.79 66.04 90)
+    (property "Reference" "R8" (at 226.06 66.04 90)
       (effects (font (size 1.27 1.27)))
     )
-    (property "Value" "470" (at 224.79 68.58 90)
+    (property "Value" "470" (at 226.06 68.58 90)
       (effects (font (size 1.27 1.27)))
     )
-    (property "Footprint" "Resistor_SMD:R_0603_1608Metric_Pad0.98x0.95mm_HandSolder" (at 224.79 70.358 90)
-      (effects (font (size 1.27 1.27)) hide)
-    )
-    (property "Datasheet" "~" (at 224.79 68.58 0)
-      (effects (font (size 1.27 1.27)) hide)
-    )
+    (property "Footprint" "Resistor_SMD:R_0603_1608Metric_Pad0.98x0.95mm_HandSolder" (at 226.06 70.358 90)
+      (effects (font (size 1.27 1.27)) hide)
+    )
+    (property "Datasheet" "~" (at 226.06 68.58 0)
+      (effects (font (size 1.27 1.27)) hide)
+    )

Commit message: ruuditud v1
Connections:
- net +3V3: no longer R17.2, U6.1 (VDD)
- net +5V: now also R17.2, U6.1 (VDD)
- net D+: now also D2.3 (I/O2); no longer D2.2 (I/O1)
- net D-: now also D2.2 (I/O1); no longer D2.3 (I/O2)
- net DIR_MINUTE: now also U4.32 (IO39); no longer U4.35 (IO42)
- net M0_MINUTE: now also U4.35 (IO42); no longer U4.32 (IO39)
- net M1_MINUTE: now also U4.34 (IO41); no longer U4.33 (IO40)
- net SEL0: now also U4.19 (IO11); no longer U4.17 (IO9)
- net SEL2: now also U4.17 (IO9); no longer U4.19 (IO11)
- net STEP_MINUTE: now also U4.33 (IO40); no longer U4.34 (IO41)

Commit message: pisibi valma???
Connections:
- net +3V3: now also R17.2, U6.1 (VDD)
- net +5V: no longer R17.2, U6.1 (VDD)
- net DIR_HOUR: now also U4.21 (IO13); no longer U4.28 (IO35)
- net DIR_MINUTE: now also U4.25 (IO48); no longer U4.32 (IO39)
- net HALL_HOUR: now also U4.20 (IO12); no longer U4.4 (IO4)
- net HALL_MINUTE: now also U4.38 (IO2); no longer U4.5 (IO5)
- net M0_HOUR: now also U4.24 (IO47); no longer U4.31 (IO38)
- net M0_MINUTE: now also U4.30 (IO37); no longer U4.35 (IO42)
- net M1_HOUR: now also U4.23 (IO21); no longer U4.30 (IO37)
- net M1_MINUTE: now also U4.29 (IO36); no longer U4.34 (IO41)
- net SEL0: now also U4.33 (IO40); no longer U4.19 (IO11)
- net SEL1: now also U4.32 (IO39); no longer U4.18 (IO10)
- net SEL2: now also U4.31 (IO38); no longer U4.17 (IO9)
- net SEL3: now also U4.34 (IO41); no longer U4.20 (IO12)
- net SERVO_PWM: now also U4.35 (IO42); no longer U4.21 (IO13)
- net STEP_HOUR: now also U4.22 (IO14); no longer U4.29 (IO36)
- net STEP_MINUTE: now also U4.28 (IO35); no longer U4.33 (IO40)
