File: skeem/servo.kicad_sch (KiCad schematic)
At the start: 9 parts, among them J10 Conn_01x03_Pin, U2 74HCT4851, U6 74HCT4851, U7 74LVC2G53

Commit message: power mgmt
Other:
- note removed: "KAS NEED SUUDAVAD PIISAVALT VOOLU V2LJA ANDA?"
- moved on the sheet: R4, R5, R6, R7, R8, U2, U6, U7

Commit message: arendus
Changed lines of the file:
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@@
     (stroke (width 0) (type default))
   )
-  (wire (pts (xy 78.74 43.18) (xy 90.17 43.18))
-    (stroke (width 0) (type default))
-  )
-  (wire (pts (xy 83.82 87.63) (xy 90.17 87.63))
+  (wire (pts (xy 87.63 43.18) (xy 90.17 43.18))
+    (stroke (width 0) (type default))
+  )
+  (wire (pts (xy 87.63 87.63) (xy 90.17 87.63))
     (stroke (width 0) (type default))
   )
@@
     (stroke (width 0) (type default))
   )
-  (wire (pts (xy 83.82 91.44) (xy 90.17 91.44))
-    (stroke (width 0) (type default))
-  )
-  (wire (pts (xy 78.74 46.99) (xy 90.17 46.99))
+  (wire (pts (xy 87.63 91.44) (xy 90.17 91.44))
+    (stroke (width 0) (type default))
+  )
+  (wire (pts (xy 87.63 46.99) (xy 90.17 46.99))
     (stroke (width 0) (type default))
   )
@@
     (stroke (width 0) (type default))
   )
-  (wire (pts (xy 78.74 50.8) (xy 90.17 50.8))
+  (wire (pts (xy 87.63 50.8) (xy 90.17 50.8))
     (stroke (width 0) (type default))
   )
@@
     (effects (font (size 1.27 1.27)) (justify right bottom))
   )
-  (hierarchical_label "SEL3" (shape input) (at 78.74 50.8 180) (fields_autoplaced)
+  (hierarchical_label "SEL3" (shape input) (at 87.63 50.8 180) (fields_autoplaced)
     (effects (font (size 1.27 1.27)) (justify right))
   )
@@
     (effects (font (size 1.27 1.27)) (justify right))
   )
-  (hierarchical_label "SEL2" (shape input) (at 83.82 91.44 180) (fields_autoplaced)
+  (hierarchical_label "SEL2" (shape input) (at 87.63 91.44 180) (fields_autoplaced)
     (effects (font (size 1.27 1.27)) (justify right))
   )
@@
     (effects (font (size 1.27 1.27)) (justify right))
   )
-  (hierarchical_label "SEL2" (shape input) (at 78.74 46.99 180) (fields_autoplaced)
+  (hierarchical_label "SEL2" (shape input) (at 87.63 46.99 180) (fields_autoplaced)
     (effects (font (size 1.27 1.27)) (justify right))
   )
-  (hierarchical_label "SEL1" (shape input) (at 78.74 43.18 180) (fields_autoplaced)
+  (hierarchical_label "SEL1" (shape input) (at 87.63 43.18 180) (fields_autoplaced)
     (effects (font (size 1.27 1.27)) (justify right))
   )
-  (hierarchical_label "SEL1" (shape input) (at 83.82 87.63 180) (fields_autoplaced)
+  (hierarchical_label "SEL1" (shape input) (at 87.63 87.63 180) (fields_autoplaced)
     (effects (font (size 1.27 1.27)) (justify right))
   )
@@
       (effects (font (size 1.27 1.27)) hide)
     )
-    (property "Datasheet" "https://4donline.ihs.com/images/VipMasterIC/IC/NEXP/NEXP-S-A0003513309/NEXP-S-A0003513309-1.pdf" (at 59.69 48.26 0)
-      (effects (font (size 1.27 1.27)) hide)
-    )
+    (property "Datasheet" "https://4donline.ihs.com/images/VipMasterIC/IC/NEXP/NEXP-S-A0003513309/NEXP-S-A0003513309-1.pdf?hkey=52A5661711E402568146F3353EA87419" (at 59.69 48.26 0)
+      (effects (font (size 1.27 1.27)) hide)
+    )

Commit message: nu and impruvd
Parts:
- removed R4, R5, R6: R, symbol Device:R
- R7, R8: value R -> 1k
Connections:
- net GND: now also U7.2 (~{EN})
Other:
- note added: "Servo pin headers"
- note removed: "Servo pin headers and current amplification"

Commit message: veel skeemi
Parts:
- added J10 (x11): Conn_01x03_Pin, Connector_PinHeader_2.54mm:PinHeader_1x03_P2.54mm_Vertical, symbol Connector:Conn_01x03_Pin
Connections:
- net +5V: now also J10.1 (Pin_1), J10.1 (Pin_1), J10.1 (Pin_1), J10.1 (Pin_1), J10.1 (Pin_1), J10.1 (Pin_1), J10.1 (Pin_1), J10.1 (Pin_1), J10.1 (Pin_1), J10.1 (Pin_1), J10.1 (Pin_1)
- net GND: now also J10.2 (Pin_2), J10.2 (Pin_2), J10.2 (Pin_2), J10.2 (Pin_2), J10.2 (Pin_2), J10.2 (Pin_2), J10.2 (Pin_2), J10.2 (Pin_2), J10.2 (Pin_2), J10.2 (Pin_2), J10.2 (Pin_2)
- net SERVO1: now also J10.3 (Pin_3)
- net SERVO10: now also J10.3 (Pin_3)
- net SERVO11: now also J10.3 (Pin_3)
- net SERVO2: now also J10.3 (Pin_3)
- net SERVO3: now also J10.3 (Pin_3)
- net SERVO4: now also J10.3 (Pin_3)
- net SERVO5: now also J10.3 (Pin_3)
- net SERVO6: now also J10.3 (Pin_3)
- net SERVO7: now also J10.3 (Pin_3)
- net SERVO8: now also J10.3 (Pin_3)
- net SERVO9: now also J10.3 (Pin_3)

Commit message: skeem
Parts:
- added C15, C16, C17: 100n, symbol Device:C
- U?: renamed from U2; footprint (none) -> Package_SO:SO-16_3.9x9.9mm_P1.27mm
- U?: renamed from U7; footprint (none) -> Package_SO:TSSOP-8_3x3mm_P0.65mm
- U?: renamed from U6; footprint (none) -> Package_SO:SO-16_3.9x9.9mm_P1.27mm
- renumbered J10 to J?, R8 to R?, R7 to R?
Connections:
- net +3V3: now also C16.1
- net +5V: now also C15.1, C17.1
- net GND: now also C15.2, C16.2, C17.2
- net MUX0_OUT1: now reaches R?.1, U?.3 (Z), U?.6 (Y1)
- net MUX0_OUT0: now reaches R?.1, U?.3 (Z), U?.7 (Y0)
Other:
- moved on the sheet: R?, U?

Commit message: skeem
Connections:
- net GND: now also U?.6 (~{EN}), U?.6 (~{EN}), U?.8 (GND), U?.8 (GND); no longer U?. (~{EN}), U?. (~{EN})
Other:
- moved on the sheet: C15, C16, C17, J?, R?, U?

Commit message: skeem
Parts:
- R? (x2): footprint (none) -> Resistor_SMD:R_0603_1608Metric_Pad0.98x0.95mm_HandSolder
Changed lines of the file:
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@@
       (effects (font (size 1.27 1.27)))
     )
-    (property "Footprint" "" (at 85.852 102.87 90)
+    (property "Footprint" "Resistor_SMD:R_0603_1608Metric_Pad0.98x0.95mm_HandSolder" (at 85.852 102.87 90)
       (effects (font (size 1.27 1.27)) hide)
     )
@@
       (effects (font (size 1.27 1.27)))
     )
-    (property "Footprint" "" (at 85.852 58.42 90)
-      (effects (font (size 1.27 1.27)) hide)
-    )
+    (property "Footprint" "Resistor_SMD:R_0603_1608Metric_Pad0.98x0.95mm_HandSolder" (at 85.852 58.42 90)
+      (effects (font (size 1.27 1.27)) hide)
+    )
