File: skeem/Stepper.kicad_sch (KiCad schematic)
At the start: 7 parts, among them J3 JST XH 5 pin, M1 Stepper_hour, M1 Stepper_minute, U6 DRV8428, U7 DRV8428

Commit message: power mgmt
Other:
- moved on the sheet: U6, U7
Changed lines of the file:
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@@
     (stroke (width 0) (type default))
   )
-  (wire (pts (xy 67.31 29.21) (xy 78.74 29.21))
+  (wire (pts (xy 50.8 24.13) (xy 62.23 24.13))
     (stroke (width 0) (type default))
   )
@@
     (stroke (width 0) (type default))
   )
-  (wire (pts (xy 67.31 33.02) (xy 78.74 33.02))
+  (wire (pts (xy 50.8 27.94) (xy 62.23 27.94))
     (stroke (width 0) (type default))
   )
@@
     (stroke (width 0) (type default))
   )
-  (wire (pts (xy 67.31 44.45) (xy 78.74 44.45))
+  (wire (pts (xy 50.8 39.37) (xy 62.23 39.37))
     (stroke (width 0) (type default))
   )
-  (wire (pts (xy 67.31 40.64) (xy 78.74 40.64))
+  (wire (pts (xy 50.8 35.56) (xy 62.23 35.56))
     (stroke (width 0) (type default))
   )
@@
     (effects (font (size 1.27 1.27)) (justify left bottom))
   )
-  (text "KAS SEE ON 6iGE?" (at 69.85 36.83 0)
+  (text "KAS SEE ON 6iGE?" (at 53.34 31.75 0)
     (effects (font (size 1.27 1.27)) (justify left bottom))
   )
@@
     (effects (font (size 1.27 1.27)) (justify left bottom))
   )
-  (label "M1_YELLOW" (at 78.74 40.64 180) (fields_autoplaced)
+  (label "M1_YELLOW" (at 62.23 35.56 180) (fields_autoplaced)
     (effects (font (size 1.27 1.27)) (justify right bottom))
   )
@@
     (effects (font (size 1.27 1.27)) (justify left bottom))
   )
-  (label "M1_PINK" (at 78.74 29.21 180) (fields_autoplaced)
+  (label "M1_PINK" (at 62.23 24.13 180) (fields_autoplaced)
     (effects (font (size 1.27 1.27)) (justify right bottom))
   )
@@
     (effects (font (size 1.27 1.27)) (justify left bottom))
   )
-  (label "M1_ORANGE" (at 78.74 33.02 180) (fields_autoplaced)
+  (label "M1_ORANGE" (at 62.23 27.94 180) (fields_autoplaced)
     (effects (font (size 1.27 1.27)) (justify right bottom))
   )
@@
     (effects (font (size 1.27 1.27)) (justify left bottom))
   )
-  (label "M1_BLUE" (at 78.74 44.45 180) (fields_autoplaced)
+  (label "M1_BLUE" (at 62.23 39.37 180) (fields_autoplaced)
     (effects (font (size 1.27 1.27)) (justify right bottom))
   )
@@
   )
   (symbol (lib_id "RVP_TopeltKell:DRV8428") (at 26.67 21.59 0) (unit 1)
-    (in_bom yes) (on_board yes) (dnp no) (fields_autoplaced)
-    (property "Reference" "U6" (at 52.07 20.32 0)
+    (in_bom yes) (on_board yes) (dnp no)
+    (property "Reference" "U6" (at 27.94 20.32 0)
       (effects (font (size 1.27 1.27)))
     )
-    (property "Value" "DRV8428" (at 52.07 22.86 0)
+    (property "Value" "DRV8428" (at 44.45 20.32 0)
       (effects (font (size 1.27 1.27)))
     )

Commit message: arendus
Parts:
- removed C3: C, symbol Device:C
- added C14: 470n, symbol Device:C
- added C15: 100n, symbol Device:C
- added C16: 10u, symbol Device:C_Polarized
- added R13, R14: 10k, symbol Device:R
Connections:
- net +5V: now reaches U6.1 (VM)
- net +5V: now also U6.15 (EN/nFAULT), U6.16 (nSLEEP), C15.2, C16.1, R13.1
- net GND: now reaches U6.11 (DECAY/TOFF)
- net GND: now also U6.2 (GND), U6.7 (GND), C14.1, C15.1, C16.2, R14.2
- net STEP_HOUR: now reaches U6.13 (STEP)
- net DIR_HOUR: now reaches U6.14 (DIR)
- net at U6.8 (DVDD): now also C14.2
- net at U6.9 (VREF): now also R13.2, R14.1
- no-connect marks 2 -> 4
Other:
- note added: "28BYJ-48 on tegelt unipolar motor, aga kui 1 pin yhendamata j2tta, pidi muutuma bipolariks..."
- note added: "Connect a X7R, 0.47-μF to 1-μF, 6.3-V or 10-V rated ceramic capacitor to GND."
- note added: "One X7R, 0.01-μF, VM-rated ceramic capacitor"
- note added: "Resistor to limit chopping current. It is recommended that the value of parallel combination of RREF1 and RREF2 should be less than 50-kΩ."
- note added: "Step angle: 5.625 x 1/64 s.t 4096 steps per revolution ~56.89 steps per 5 deg"
- note added: "internal pulldown"
- note added: "kas vajame microsteppingut? internal pulldown"
- moved on the sheet: U6, U7

Commit message: nu and impruvd
Parts:
- R13: value 10k -> 27k
- R14: value 10k -> 5k
Connections:
- net DIR_MINUTE: now also U7.14 (DIR)
- net STEP_MINUTE: now also U7.13 (STEP)
- net M0_HOUR: now reaches U6.10 (M0)
- net M1_HOUR: now reaches U6.12 (M1)
- net M0_MINUTE: now reaches U7.10 (M0)
- net M1_MINUTE: now reaches U7.12 (M1)
- no-connect marks 4 -> 2
Other:
- note added: "28BYJ-48 on tegelt unipolar motor, aga kui 1 trace l2bi l6igata, saab muuta bipolariks"
- note added: "BYJ28-48 5V motor winding resistance 50R i.e nom current 100 mA but when converted to bipolar winding resistance doubles therefore current should double as well?"
- note added: "I = VREF / 3 27k and 5k yields ~0.8V VREF and motor crrent of 260mA"
- note added: "äkki panna kruviga smd potekas?"
- note removed: "28BYJ-48 on tegelt unipolar motor, aga kui 1 pin yhendamata j2tta, pidi muutuma bipolariks..."
- moved on the sheet: C14, C15, C16, J3, M1, R13, R14, U6, U7

Commit message: veel skeemi
Parts:
- removed M1: Stepper_minute, symbol Motor:Stepper_Motor_bipolar
- removed M1: Stepper_hour, symbol Motor:Stepper_Motor_bipolar
- added C1: 10u, symbol Device:C_Polarized
- added C19: 10n, symbol Device:C
- added C20: 470n, symbol Device:C
- added R16: 33k, symbol Device:R
- added R17: 5k1, symbol Device:R
- added RV1, RV2: 1M, symbol Device:R_Potentiometer
- C15: value 100n -> 10n
- R13: value 27k -> 33k
- R14: value 5k -> 5k1
Connections:
- net M2_BLUE is gone; now on net M2_A1: J3.1 (Pin_1)
- net M2_ORANGE is gone; now on net M2_B2: J3.4 (Pin_4)
- net M2_PINK is gone; now on net M2_B1: J3.2 (Pin_2)
- net M2_YELLOW is gone; now on net M2_A2: J3.3 (Pin_3)
- net +5V: now also U7.15 (EN/nFAULT), U7.16 (nSLEEP), RV1.1, RV2.1; no longer C15.2, C16.1, R13.1, U6.1 (VM)
- net GND: now also U7.11 (DECAY/TOFF), U7.2 (GND), U7.7 (GND), C1.2, C19.1, C20.1, R17.2
- net +9V: now reaches U7.1 (VM)
- net +9V: now also C15.2, C16.1, U6.1 (VM), C1.1, C19.2
- net M2_A1: now reaches U7.3 (AOUT1)
- net M2_A2: now reaches U7.4 (AOUT2)
- net M2_B2: now reaches U7.5 (BOUT2)
- net M2_B1: now reaches U7.6 (BOUT1)
- net at U7.8 (DVDD): now also C20.2
- net at U7.9 (VREF): now also R16.2, R17.1
- net M1_BLUE renamed M1_A1
- net M1_A1: now also U6.3 (AOUT1); no longer U6.5 (BOUT2)
- net M1_ORANGE renamed M1_A2
- net M1_A2: now also J3.3 (Pin_3); no longer J3.4 (Pin_4)
- net M1_PINK renamed M1_B1
- net M1_B1: now also U6.6 (BOUT1); no longer U6.3 (AOUT1)
- removed net M1_YELLOW: J3.3 (Pin_3), U6.6 (BOUT1)
- new net: R16.1, RV2.2
- new net: R13.1, RV1.2
- new net M1_B2: J3.4 (Pin_4), U6.5 (BOUT2)
- no-connect marks 2 -> 4
Other:
- note added: "BYJ28-48 5V motor winding resistance 40R max current 9V/40R = 225mA i.e max current VREF 0.225*3=0.675V"
- note added: "IFS (A) = VREF (V) / 3 (V/A)"
- note added: "Step angle: 5.625 x 1/64 i.e 4096 steps per revolution ~56.89 steps per 5 deg"
- note added: "VREF max 5 * (5.1/38.1) = 0.670 V VREF min 5 * (5.1/1038.1) = 0.025 V which yields 8 mA motor current"
- note added: "winding 1 blue and yellow wires winding 2 pink and orange wires"
- note removed: "28BYJ-48 on tegelt unipolar motor, aga kui 1 trace l2bi l6igata, saab muuta bipolariks"
- note removed: "BYJ28-48 5V motor winding resistance 50R i.e nom current 100 mA but when converted to bipolar winding resistance doubles therefore current should double as well?"
- note removed: "I = VREF / 3 27k and 5k yields ~0.8V VREF and motor crrent of 260mA"
- note removed: "KAS SEE ON 6iGE?"
- note removed: "Step angle: 5.625 x 1/64 s.t 4096 steps per revolution ~56.89 steps per 5 deg"
- note removed: "internal pulldown"
- note removed: "kas vajame microsteppingut? internal pulldown"
- note removed: "äkki panna kruviga smd potekas?"
- moved on the sheet: J3, R13, U7

Commit message: skeem
Parts:
- J? (x2): renamed from J3; footprint (none) -> Connector_JST:JST_XH_B5B-XH-A_1x05_P2.50mm_Vertical
- U8: renamed from U6; footprint (none) -> Package_SO:HTSSOP-16-1EP_4.4x5mm_P0.65mm_EP3x3mm
- U9: renamed from U7; footprint (none) -> Package_SO:HTSSOP-16-1EP_4.4x5mm_P0.65mm_EP3x3mm
- renumbered C16 to C18, C15 to C19, C14 to C20, C1 to C21, C19 to C22, C20 to C23, R13 to R16, R14 to R17, R16 to R18, R17 to R19

Commit message: skeem
Other:
- note added: "BYJ28-48 5V motor winding resistance 40R max current 9V/40R = 225mA i.e max current VREF 0.225*3 = 0.675V"
- note added: "VREF max 5 * (5.1/38.1) = 0.670V VREF min 5 * (5.1/1038.1) = 0.025V which yields 8 mA motor current"
- note added: "osta korralik potekas"
- note removed: "BYJ28-48 5V motor winding resistance 40R max current 9V/40R = 225mA i.e max current VREF 0.225*3=0.675V"
- note removed: "VREF max 5 * (5.1/38.1) = 0.670 V VREF min 5 * (5.1/1038.1) = 0.025 V which yields 8 mA motor current"
Changed lines of the file:
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@@
   (junction (at 96.52 25.4) (diameter 0) (color 0 0 0 0)
   )
+  (junction (at 113.03 124.46) (diameter 0) (color 0 0 0 0)
+  )
   (junction (at 110.49 25.4) (diameter 0) (color 0 0 0 0)
   )
@@
   )
   (junction (at 113.03 40.64) (diameter 0) (color 0 0 0 0)
+  )
+  (junction (at 113.03 33.02) (diameter 0) (color 0 0 0 0)
   )
   (junction (at 96.52 124.46) (diameter 0) (color 0 0 0 0)
@@
     (stroke (width 0) (type default))
   )
+  (wire (pts (xy 113.03 124.46) (xy 115.57 124.46))
+    (stroke (width 0) (type default))
+  )
   (wire (pts (xy 142.24 29.21) (xy 153.67 29.21))
     (stroke (width 0) (type default))
@@
     (stroke (width 0) (type default))
   )
-  (wire (pts (xy 110.49 33.02) (xy 115.57 33.02))
+  (wire (pts (xy 110.49 33.02) (xy 113.03 33.02))
     (stroke (width 0) (type default))
   )
@@
     (stroke (width 0) (type default))
   )
-  (wire (pts (xy 110.49 124.46) (xy 115.57 124.46))
+  (wire (pts (xy 110.49 124.46) (xy 113.03 124.46))
     (stroke (width 0) (type default))
   )
@@
   )
   (wire (pts (xy 110.49 25.4) (xy 115.57 25.4))
+    (stroke (width 0) (type default))
+  )
+  (wire (pts (xy 113.03 33.02) (xy 115.57 33.02))
     (stroke (width 0) (type default))
   )
@@
   )
   (text "Connect a X7R, 0.47-μF to 1-μF, 6.3-V\nor 10-V rated ceramic capacitor to GND."
-    (at 36.83 34.29 0)
-    (effects (font (size 1.27 1.27)) (justify left bottom))
-  )
-  (text "VREF max 5 * (5.1/38.1) = 0.670 V\nVREF min 5 * (5.1/1038.1) = 0.025 V \nwhich yields 8 mA motor current\n"
+    (at 31.75 34.29 0)
+    (effects (font (size 1.27 1.27)) (justify left bottom))
+  )
+  (text "VREF max 5 * (5.1/38.1) = 0.670V\nVREF min 5 * (5.1/1038.1) = 0.025V \nwhich yields 8 mA motor current\n"
     (at 21.59 96.52 0)
     (effects (font (size 1.27 1.27)) (justify left bottom))
   )
-  (text "One X7R, 0.01-μF, VM-rated ceramic capacitor" (at 36.83 25.4 0)
+  (text "One X7R, 0.01-μF, VM-rated ceramic capacitor" (at 31.75 25.4 0)
     (effects (font (size 1.27 1.27)) (justify left bottom))
   )
@@
     (effects (font (size 2.032 2.032)) (justify left bottom))
   )
-  (text "BYJ28-48 5V motor\nwinding resistance 40R\nmax current 9V/40R = 225mA\ni.e max current VREF 0.225*3=0.675V"
+  (text "BYJ28-48 5V motor\nwinding resistance 40R\nmax current 9V/40R = 225mA\ni.e max current VREF 0.225*3 = 0.675V"
     (at 21.59 85.09 0)
     (effects (font (size 1.27 1.27)) (justify left bottom))
@@
     (effects (font (size 1.27 1.27)) (justify left bottom))
   )
+  (text "osta korralik potekas" (at 72.39 88.9 0)
+    (effects (font (size 1.27 1.27)) (justify left bottom))
+  )
   (label "M1_B1" (at 153.67 36.83 180) (fields_autoplaced)
     (effects (font (size 1.27 1.27)) (justify right bottom))
@@
   (hierarchical_label "DIR_HOUR" (shape input) (at 107.95 52.07 180) (fields_autoplaced)
     (effects (font (size 1.27 1.27)) (justify right))
+  )
+  (symbol (lib_id "power:PWR_FLAG") (at 113.03 33.02 0) (unit 1)
+    (in_bom yes) (on_board yes) (dnp no) (fields_autoplaced)
+    (property "Reference" "#FLG02" (at 113.03 31.115 0)
+      (effects (font (size 1.27 1.27)) hide)
+    )
+    (property "Value" "PWR_FLAG" (at 113.03 27.94 0)
+      (effects (font (size 1.27 1.27)) hide)
+    )
+    (property "Footprint" "" (at 113.03 33.02 0)
+      (effects (font (size 1.27 1.27)) hide)
+    )
+    (property "Datasheet" "~" (at 113.03 33.02 0)
+      (effects (font (size 1.27 1.27)) hide)
+    )
+    (pin "1")
+    (instances
+      (project "RVP_TopeltKell"
+        (path "/55c41515-c5b3-46de-9fdd-e6e788e90361"
+          (reference "#FLG02") (unit 1)
+        )
+        (path "/55c41515-c5b3-46de-9fdd-e6e788e90361/73cb924a-5bea-4e51-900c-7d71494886f5"
+          (reference "#FLG05") (unit 1)
+        )
+      )
+    )
   )
   (symbol (lib_id "power:+5V") (at 91.44 166.37 0) (unit 1)
@@
         )
       )
+    )
+  )
+  (symbol (lib_id "power:PWR_FLAG") (at 113.03 124.46 0) (unit 1)
+    (in_bom yes) (on_board yes) (dnp no) (fields_autoplaced)
+    (property "Reference" "#FLG02" (at 113.03 122.555 0)
+      (effects (font (size 1.27 1.27)) hide)
+    )
+    (property "Value" "PWR_FLAG" (at 113.03 119.38 0)
+      (effects (font (size 1.27 1.27)) hide)
+    )
+    (property "Footprint" "" (at 113.03 124.46 0)
+      (effects (font (size 1.27 1.27)) hide)
+    )
+    (property "Datasheet" "~" (at 113.03 124.46 0)
+      (effects (font (size 1.27 1.27)) hide)
+    )
+    (pin "1")
+    (instances
+      (project "RVP_TopeltKell"
+        (path "/55c41515-c5b3-46de-9fdd-e6e788e90361"
+          (reference "#FLG02") (unit 1)
+        )
+        (path "/55c41515-c5b3-46de-9fdd-e6e788e90361/73cb924a-5bea-4e51-900c-7d71494886f5"
+          (reference "#FLG04") (unit 1)
+        )
+      )

Commit message: skeem
Parts:
- R16, R17, R18, R19: footprint (none) -> Resistor_SMD:R_0603_1608Metric_Pad0.98x0.95mm_HandSolder
Changed lines of the file:
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@@
       (effects (font (size 1.27 1.27)))
     )
-    (property "Footprint" "" (at 99.06 171.958 90)
+    (property "Footprint" "Resistor_SMD:R_0603_1608Metric_Pad0.98x0.95mm_HandSolder" (at 99.06 171.958 90)
       (effects (font (size 1.27 1.27)) hide)
     )
@@
       (effects (font (size 1.27 1.27)) (justify left))
     )
-    (property "Footprint" "" (at 101.092 82.55 90)
+    (property "Footprint" "Resistor_SMD:R_0603_1608Metric_Pad0.98x0.95mm_HandSolder" (at 101.092 82.55 90)
       (effects (font (size 1.27 1.27)) hide)
     )
@@
       (effects (font (size 1.27 1.27)) (justify left))
     )
-    (property "Footprint" "" (at 101.092 173.99 90)
+    (property "Footprint" "Resistor_SMD:R_0603_1608Metric_Pad0.98x0.95mm_HandSolder" (at 101.092 173.99 90)
       (effects (font (size 1.27 1.27)) hide)
     )
@@
       (effects (font (size 1.27 1.27)))
     )
-    (property "Footprint" "" (at 99.06 80.518 90)
-      (effects (font (size 1.27 1.27)) hide)
-    )
+    (property "Footprint" "Resistor_SMD:R_0603_1608Metric_Pad0.98x0.95mm_HandSolder" (at 99.06 80.518 90)
+      (effects (font (size 1.27 1.27)) hide)
+    )

Commit message: pcb comp placement draft
Parts:
- removed C18, C21: 10u, symbol Device:C_Polarized
- removed R16, R18: 33k, Resistor_SMD:R_0603_1608Metric_Pad0.98x0.95mm_HandSolder, symbol Device:R
- removed R17, R19: 5k1, Resistor_SMD:R_0603_1608Metric_Pad0.98x0.95mm_HandSolder, symbol Device:R
- removed RV2: 1M, symbol Device:R_Potentiometer
- added C22, C25: 10u, Capacitor_SMD:C_0805_2012Metric_Pad1.18x1.45mm_HandSolder, symbol Device:C
- added R20: 10k, Resistor_SMD:R_0603_1608Metric_Pad0.98x0.95mm_HandSolder, symbol Device:R
- C23: renamed from C19; footprint (none) -> Capacitor_SMD:C_0603_1608Metric_Pad1.08x0.95mm_HandSolder
- C24: renamed from C20; footprint (none) -> Capacitor_SMD:C_0603_1608Metric_Pad1.08x0.95mm_HandSolder
- C26: renamed from C22; footprint (none) -> Capacitor_SMD:C_0603_1608Metric_Pad1.08x0.95mm_HandSolder
- C27: renamed from C23; footprint (none) -> Capacitor_SMD:C_0603_1608Metric_Pad1.08x0.95mm_HandSolder
- RV1: value 1M -> 1k; footprint (none) -> Potentiometer_THT:Potentiometer_Bourns_3386P_Vertical
- renumbered U8 to U10, U9 to U11
Connections:
- net +5V: now also R20.1; no longer RV1.1
- net +9V: now also C22.1, C25.1
- net GND: now also RV1.3, C22.2, C25.2
- net VREF: now reaches U11.9 (VREF)
- net VREF: now also RV1.2, U10.9 (VREF)
- new net: R20.2, RV1.1
- no-connect marks 4 -> 2
Other:
- note added: "VREF max 5 * (1/11) = 0.45V VREF min 5 * (0/11) = 0V Imotor max 150 mA"
- note removed: "VREF max 5 * (5.1/38.1) = 0.670V VREF min 5 * (5.1/1038.1) = 0.025V which yields 8 mA motor current"
- note removed: "osta korralik potekas"
