File: skeem/Stepper.kicad_sch (KiCad schematic)
At the start: 12 parts, among them U10 DRV8428, U11 DRV8428

Commit message: natuke pcbd
Parts:
- added C16 (x2): 100n, Capacitor_SMD:C_0603_1608Metric_Pad1.08x0.95mm_HandSolder, symbol Device:C
Connections:
- net GND: now also C16.2, C16.2
- net M1_A1: now also J?.4 (Pin_4); no longer J?.1 (Pin_1)
- net M1_B1: now also J?.1 (Pin_1); no longer J?.2 (Pin_2)
- net M1_B2: now also J?.2 (Pin_2); no longer J?.4 (Pin_4)
- net M2_A1: now also J?.4 (Pin_4); no longer J?.1 (Pin_1)
- net M2_B1: now also J?.1 (Pin_1); no longer J?.2 (Pin_2)
- net M2_B2: now also J?.2 (Pin_2); no longer J?.4 (Pin_4)
- net VREF: now also C16.1, C16.1
Changed lines of the file:
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@@
     (effects (font (size 1.27 1.27)) (justify right bottom))
   )
-  (label "M1_B2" (at 184.15 36.83 0) (fields_autoplaced)
+  (label "M1_B2" (at 184.15 31.75 0) (fields_autoplaced)
     (effects (font (size 1.27 1.27)) (justify left bottom))
   )
@@
     (effects (font (size 1.27 1.27)) (justify left bottom))
   )
-  (label "M2_B1" (at 175.26 121.92 0) (fields_autoplaced)
+  (label "M2_B1" (at 175.26 119.38 0) (fields_autoplaced)
     (effects (font (size 1.27 1.27)) (justify left bottom))
   )
@@
     (effects (font (size 1.27 1.27)) (justify left bottom))
   )
-  (label "M2_A1" (at 175.26 119.38 0) (fields_autoplaced)
+  (label "M2_A1" (at 175.26 127 0) (fields_autoplaced)
     (effects (font (size 1.27 1.27)) (justify left bottom))
   )
@@
     (effects (font (size 1.27 1.27)) (justify right bottom))
   )
-  (label "M1_A1" (at 184.15 29.21 0) (fields_autoplaced)
+  (label "M1_A1" (at 184.15 36.83 0) (fields_autoplaced)
     (effects (font (size 1.27 1.27)) (justify left bottom))
   )
@@
     (effects (font (size 1.27 1.27)) (justify right bottom))
   )
-  (label "M2_B2" (at 175.26 127 0) (fields_autoplaced)
-    (effects (font (size 1.27 1.27)) (justify left bottom))
-  )
-  (label "M1_B1" (at 184.15 31.75 0) (fields_autoplaced)
+  (label "M2_B2" (at 175.26 121.92 0) (fields_autoplaced)
+    (effects (font (size 1.27 1.27)) (justify left bottom))
+  )
+  (label "M1_B1" (at 184.15 29.21 0) (fields_autoplaced)
     (effects (font (size 1.27 1.27)) (justify left bottom))
   )
@@
         (path "/55c41515-c5b3-46de-9fdd-e6e788e90361/73cb924a-5bea-4e51-900c-7d71494886f5"
           (reference "#PWR081") (unit 1)
+        )
+      )
+    )
+  )
+  (symbol (lib_id "power:GND") (at 105.41 86.36 0) (unit 1)
+    (in_bom yes) (on_board yes) (dnp no) (fields_autoplaced)
+    (property "Reference" "#PWR093" (at 105.41 92.71 0)
+      (effects (font (size 1.27 1.27)) hide)
+    )
+    (property "Value" "GND" (at 105.41 91.44 0)
+      (effects (font (size 1.27 1.27)) hide)
+    )
+    (property "Footprint" "" (at 105.41 86.36 0)
+      (effects (font (size 1.27 1.27)) hide)
+    )
+    (property "Datasheet" "" (at 105.41 86.36 0)
+      (effects (font (size 1.27 1.27)) hide)
+    )
+    (pin "1")
+    (instances
+      (project "RVP_TopeltKell"
+        (path "/55c41515-c5b3-46de-9fdd-e6e788e90361/73cb924a-5bea-4e51-900c-7d71494886f5"
+          (reference "#PWR093") (unit 1)
         )
       )
@@
     )
   )
+  (symbol (lib_id "Device:C") (at 105.41 82.55 0) (unit 1)
+    (in_bom yes) (on_board yes) (dnp no) (fields_autoplaced)
+    (property "Reference" "C16" (at 109.22 81.28 0)
+      (effects (font (size 1.27 1.27)) (justify left))
+    )
+    (property "Value" "100n" (at 109.22 83.82 0)
+      (effects (font (size 1.27 1.27)) (justify left))
+    )
+    (property "Footprint" "Capacitor_SMD:C_0603_1608Metric_Pad1.08x0.95mm_HandSolder" (at 106.3752 86.36 0)
+      (effects (font (size 1.27 1.27)) hide)
+    )
+    (property "Datasheet" "~" (at 105.41 82.55 0)
+      (effects (font (size 1.27 1.27)) hide)
+    )
+    (pin "1")
+    (pin "2")
+    (instances
+      (project "RVP_TopeltKell"
+        (path "/55c41515-c5b3-46de-9fdd-e6e788e90361"
+          (reference "C16") (unit 1)
+        )
+        (path "/55c41515-c5b3-46de-9fdd-e6e788e90361/73cb924a-5bea-4e51-900c-7d71494886f5"
+          (reference "C29") (unit 1)
+        )
+      )
+    )
+  )
   (symbol (lib_id "power:GND") (at 87.63 82.55 0) (unit 1)
     (in_bom yes) (on_board yes) (dnp no) (fields_autoplaced)
@@
     )
   )
+  (symbol (lib_id "power:GND") (at 105.41 177.8 0) (unit 1)
+    (in_bom yes) (on_board yes) (dnp no) (fields_autoplaced)
+    (property "Reference" "#PWR029" (at 105.41 184.15 0)
+      (effects (font (size 1.27 1.27)) hide)
+    )
+    (property "Value" "GND" (at 105.41 182.88 0)
+      (effects (font (size 1.27 1.27)) hide)
+    )
+    (property "Footprint" "" (at 105.41 177.8 0)
+      (effects (font (size 1.27 1.27)) hide)
+    )
+    (property "Datasheet" "" (at 105.41 177.8 0)
+      (effects (font (size 1.27 1.27)) hide)
+    )
+    (pin "1")
+    (instances
+      (project "RVP_TopeltKell"
+        (path "/55c41515-c5b3-46de-9fdd-e6e788e90361/73cb924a-5bea-4e51-900c-7d71494886f5"
+          (reference "#PWR029") (unit 1)
+        )
+      )
+    )
+  )
   (symbol (lib_id "Device:C") (at 96.52 120.65 180) (unit 1)
     (in_bom yes) (on_board yes) (dnp no)
@@
         )
       )
+    )
+  )
+  (symbol (lib_id "Device:C") (at 105.41 173.99 0) (unit 1)
+    (in_bom yes) (on_board yes) (dnp no) (fields_autoplaced)
+    (property "Reference" "C16" (at 109.22 172.72 0)
+      (effects (font (size 1.27 1.27)) (justify left))
+    )
+    (property "Value" "100n" (at 109.22 175.26 0)
+      (effects (font (size 1.27 1.27)) (justify left))
+    )
+    (property "Footprint" "Capacitor_SMD:C_0603_1608Metric_Pad1.08x0.95mm_HandSolder" (at 106.3752 177.8 0)
+      (effects (font (size 1.27 1.27)) hide)
+    )
+    (property "Datasheet" "~" (at 105.41 173.99 0)
+      (effects (font (size 1.27 1.27)) hide)
+    )
+    (pin "1")
+    (pin "2")
+    (instances
+      (project "RVP_TopeltKell"
+        (path "/55c41515-c5b3-46de-9fdd-e6e788e90361"
+          (reference "C16") (unit 1)
+        )
+        (path "/55c41515-c5b3-46de-9fdd-e6e788e90361/73cb924a-5bea-4e51-900c-7d71494886f5"
+          (reference "C28") (unit 1)
+        )
+      )

Commit message: ruuditud v1
Connections:
- net GND: now also U10.17 (GND), U11.17 (GND)
Changed lines of the file:
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@@
+    (stroke (width 0) (type default))
+  )
+  (wire (pts (xy 134.62 83.82) (xy 134.62 86.36))
     (stroke (width 0) (type default))
   )
@@
     (stroke (width 0) (type default))
   )
+  (wire (pts (xy 134.62 177.8) (xy 134.62 175.26))
+    (stroke (width 0) (type default))
+  )
   (wire (pts (xy 142.24 25.4) (xy 153.67 25.4))
     (stroke (width 0) (type default))
@@
     (stroke (width 0) (type default))
   )
+  (wire (pts (xy 130.81 177.8) (xy 134.62 177.8))
+    (stroke (width 0) (type default))
+  )
   (wire (pts (xy 114.3 162.56) (xy 115.57 162.56))
     (stroke (width 0) (type default))
@@
   )
   (wire (pts (xy 130.81 175.26) (xy 130.81 177.8))
+    (stroke (width 0) (type default))
+  )
+  (wire (pts (xy 130.81 86.36) (xy 134.62 86.36))
     (stroke (width 0) (type default))
   )
@@
     )
   )
-  (symbol (lib_id "RVP_TopeltKell:DRV8428") (at 118.11 22.86 0) (unit 1)
+  (symbol (lib_name "DRV8428_1") (lib_id "RVP_TopeltKell:DRV8428") (at 118.11 22.86 0) (unit 1)
     (in_bom yes) (on_board yes) (dnp no)
     (property "Reference" "U10" (at 119.38 21.59 0)
@@
     (pin "15")
     (pin "16")
+    (pin "17")
     (pin "2")
     (pin "3")
@@
     (pin "15")
     (pin "16")
+    (pin "17")
     (pin "2")
     (pin "3")
